File: _autosave-05833-Project2.kicad_sch (KiCad schematic)
At the start: 13 parts, among them J1 BB Power, J2 FTDI, J3 AREF, J4 GPIO, U1 LM7805, U2 ATmega328-P, Y1 16MHz Resonator

Commit message: Updates to the edge cuts
Parts:
- renumbered J3 to AREF
Changed lines of the file:
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@@
 		(dnp no)
 		(fields_autoplaced yes)
-		(property "Reference" "J3"
+		(property "Reference" "AREF"
 			(at 88.265 45.72 0)
 			(effects
@@
 			(project "05833-Project2"
 				(path "/e30c0031-f481-430a-8ab4-08825872f914"
-					(reference "J3")
+					(reference "AREF")
 					(unit 1)
 				)
