File: Initial Project 2/05833-Project2.kicad_pcb (KiCad board)
At the start: 2 copper layers, 63 x 32 mm, 13 parts, among them J1 BB, J2 FTDI, J3 AREF, J4 GPIO, U1 LM7805, U2 ATmega328-P, Y1 16MHz Resonator

Commit message: Revamped
Parts:
- moved C4 31.1 mm to (63.0, 63.5)
- moved Y1 7.52 mm to (71.5, 63.5)
Routing:
- net Net-(U2-XTAL2/PB7): track 10.2 -> 3.83 mm
- net GND: track 146.1 -> 141.5 mm
- net Net-(U2-XTAL1/PB6): track 7.73 -> 3.95 mm
Changed lines of the file:
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@@
 	(footprint "05833:C_Disc_D3.0mm_W1.6mm_P2.50mm"
 		(layer "F.Cu")
-		(at 92.09405 52.469665 180)
+		(at 63 63.5 180)
 		(descr "C, Disc series, Radial, pin pitch=2.50mm, , diameter*width=3.0*1.6mm^2, Capacitor, http://www.vishay.com/docs/45233/krseries.pdf")
 		(tags "C Disc series Radial pin pitch 2.50mm  diameter 3.0mm width 1.6mm Capacitor")
@@
 	(footprint "05833:Resonator-3Pin_W6.0mm_H3.0mm"
 		(layer "F.Cu")
-		(at 79 64 180)
+		(at 71.5 63.5 180)
 		(descr "Ceramic Resomator/Filter 6.0x3.0mm^2, length*width=6.0x3.0mm^2 package, package length=6.0mm, package width=3.0mm, 3 pins")
 		(tags "THT ceramic resonator filter")
@@
 	)
 	(segment
-		(start 76.5 64)
-		(end 74.12 61.62)
+		(start 67.85 64.65)
+		(end 64.15 64.65)
 		(width 0.2)
 		(layer "F.Cu")
@@
 	)
 	(segment
-		(start 92.069324 56.739437)
-		(end 92.069324 60.975274)
+		(start 61.9 64.6)
+		(end 63 63.5)
 		(width 0.2)
 		(layer "F.Cu")
@@
 	)
 	(segment
-		(start 98.329121 60.475551)
-		(end 98.329121 57.983051)
+		(start 52.964365 55.7)
+		(end 49 59.664365)
 		(width 0.2)
 		(layer "F.Cu")
@@
 	)
 	(segment
-		(start 68.315635 59)
-		(end 66.46 59)
+		(start 65.34 61.16)
+		(end 65.34 60.12)
 		(width 0.2)
 		(layer "F.Cu")
@@
 	)
 	(segment
-		(start 105 72.447203)
-		(end 104.995541 72.442744)
+		(start 92.069324 56.739437)
+		(end 92.069324 60.975274)
 		(width 0.2)
 		(layer "F.Cu")
@@
 	)
 	(segment
-		(start 68.98 60.48)
-		(end 68.98 59.664365)
+		(start 98.329121 60.475551)
+		(end 98.329121 57.983051)
 		(width 0.2)
 		(layer "F.Cu")
@@
 	)
 	(segment
-		(start 92.09405 56.544598)
-		(end 92.09405 52.469665)
+		(start 105 72.447203)
+		(end 104.995541 72.442744)
 		(width 0.2)
 		(layer "F.Cu")
@@
 	)
 	(segment
-		(start 52.964365 55.7)
-		(end 49 59.664365)
-		(width 0.2)
-		(layer "F.Cu")
-		(net 2)
-	)
-	(segment
 		(start 91.4 67.404672)
 		(end 98.329121 60.475551)
@@
 	)
 	(segment
-		(start 49 60.575635)
-		(end 50.044365 61.62)
+		(start 64.15 64.65)
+		(end 63 63.5)
 		(width 0.2)
 		(layer "F.Cu")
@@
 	)
 	(segment
-		(start 105.095 72.135)
-		(end 105 72.04)
-		(width 0.2)
-		(layer "F.Cu")
-		(net 2)
-	)
-	(segment
-		(start 59.6 55.7)
-		(end 52.964365 55.7)
-		(width 0.2)
-		(layer "F.Cu")
-		(net 2)
-	)
-	(segment
-		(start 66.46 59)
-		(end 65.34 60.12)
+		(start 49 59.664365)
+		(end 49 60.575635)
 		(width 0.2)
 		(layer "F.Cu")
@@
 	)
 	(segment
-		(start 62 52.5)
-		(end 62.8 52.5)
+		(start 105.095 72.135)
+		(end 105 72.04)
 		(width 0.2)
 		(layer "F.Cu")
@@
 	)
 	(segment
-		(start 62.8 52.5)
-		(end 59.6 55.7)
+		(start 69 63.5)
+		(end 67.85 64.65)
 		(width 0.2)
 		(layer "F.Cu")
@@
 	)
 	(segment
-		(start 49 59.664365)
-		(end 49 60.575635)
+		(start 63 63.5)
+		(end 65.34 61.16)
 		(width 0.2)
 		(layer "F.Cu")
@@
 	)
 	(segment
-		(start 63.84 61.62)
-		(end 65.34 60.12)
+		(start 92 56.808761)
+		(end 92 57)
 		(width 0.2)
 		(layer "F.Cu")
@@
 	)
 	(segment
-		(start 70.12 61.62)
-		(end 68.98 60.48)
+		(start 105 77.105)
+		(end 105 76.7)
 		(width 0.2)
 		(layer "F.Cu")
@@
 	)
 	(segment
-		(start 105 77.105)
-		(end 105 76.7)
+		(start 98.329121 57.983051)
+		(end 97.029121 56.683051)
 		(width 0.2)
 		(layer "F.Cu")
@@
 	)
 	(segment
-		(start 98.329121 57.983051)
-		(end 97.029121 56.683051)
+		(start 53.024365 64.6)
+		(end 61.9 64.6)
+		(width 0.2)
+		(layer "F.Cu")
+		(net 2)
+	)
+	(segment
+		(start 49 60.575635)
+		(end 53.024365 64.6)
 		(width 0.2)
 		(layer "F.Cu")
@@
 	)
 	(segment
-		(start 50.044365 61.62)
-		(end 63.84 61.62)
+		(start 59.6 55.7)
+		(end 52.964365 55.7)
 		(width 0.2)
 		(layer "F.Cu")
@@
 	)
 	(segment
-		(start 74.12 61.62)
-		(end 70.12 61.62)
+		(start 62.8 52.5)
+		(end 59.6 55.7)
 		(width 0.2)
 		(layer "F.Cu")
@@
 	)
 	(segment
-		(start 68.98 59.664365)
-		(end 68.315635 59)
+		(start 92.069324 52.444938)
+		(end 92.062193 52.437807)
 		(width 0.2)
-		(layer "F.Cu")
+		(layer "B.Cu")
 		(net 2)
 	)
@@
 	)
 	(segment
+		(start 92.069324 56.739437)
+		(end 92.069324 52.444938)
+		(width 0.2)
+		(layer "B.Cu")
+		(net 2)
+	)
+	(segment
+		(start 92.062193 52.437807)
+		(end 89.624385 50)
+		(width 0.2)
+		(layer "B.Cu")
+		(net 2)
+	)
+	(segment
 		(start 89.624385 50)
 		(end 65.3 50)
@@
 	)
 	(segment
-		(start 104.995541 72.995541)
-		(end 105 73)
+		(start 92.09405 52.469665)
+		(end 92.062193 52.437807)
 		(width 0.2)
 		(layer "B.Cu")
@@
 	)
 	(segment
-		(start 104.995541 69.902744)
-		(end 104.995541 72.442744)
+		(start 104.995541 72.995541)
+		(end 105 73)
 		(width 0.2)
 		(layer "B.Cu")
@@
 	)
 	(segment
-		(start 92.09405 52.469665)
-		(end 89.624385 50)
+		(start 104.995541 69.902744)
+		(end 104.995541 72.442744)
 		(width 0.2)
 		(layer "B.Cu")
@@
 	)
 	(segment
-		(start 51.72 61.22)
-		(end 61.7 61.22)
+		(start 60.5 63.5)
+		(end 62.8 61.2)
 		(width 0.2)
 		(layer "F.Cu")
@@
 	)
 	(segment
-		(start 90.69405 51.369665)
-		(end 94.255735 51.369665)
-		(width 0.2)
-		(layer "F.Cu")
-		(net 3)
-	)
-	(segment
-		(start 89.59405 52.469665)
-		(end 89.59405 56.714711)
+		(start 89.569324 56.739437)
+		(end 92.16571 54.143051)
 		(width 0.2)
 		(layer "F.Cu")
@@
 	)
 	(segment
-		(start 89.59405 52.469665)
-		(end 90.69405 51.369665)
+		(start 96.569121 54.643051)
+		(end 97.029121 54.183051)
 		(width 0.2)
 		(layer "F.Cu")
@@
 	)
 	(segment
-		(start 94.255735 51.369665)
-		(end 97.029121 54.143051)
+		(start 60.5 61.22)
+		(end 61.7 61.22)
 		(width 0.2)
 		(layer "F.Cu")
@@
 	)
 	(segment
-		(start 96.569121 54.643051)
-		(end 97.029121 54.183051)
+		(start 51.72 61.22)
+		(end 60.5 61.22)
 		(width 0.2)
 		(layer "F.Cu")
@@
 	)
 	(segment
-		(start 89.59405 56.714711)
-		(end 89.569324 56.739437)
-		(width 0.2)
-		(layer "F.Cu")
-		(net 3)
-	)
-	(segment
 		(start 88.929887 56.1)
 		(end 71.48 56.1)
@@
 	)
 	(segment
+		(start 92.16571 54.143051)
+		(end 97.029121 54.143051)
+		(width 0.2)
+		(layer "F.Cu")
+		(net 3)
+	)
+	(segment
 		(start 51.5 59.704365)
 		(end 51.5 61)
@@
 	)
 	(segment
+		(start 62.8 61.2)
+		(end 62.8 60.12)
+		(width 0.2)
+		(layer "F.Cu")
+		(net 3)
+	)
+	(segment
 		(start 90.99405 63.49405)
 		(end 90.99405 58.164163)
@@
 	)
 	(segment
-		(start 72.02 62.02)
-		(end 69.78 62.02)
-		(width 0.2)
-		(layer "F.Cu")
-		(net 27)
-	)
-	(segment
-		(start 74 64)
-		(end 72.02 62.02)
+		(start 66.5 63.5)
+		(end 66.5 61.5)
 		(width 0.2)
 		(layer "F.Cu")
@@
 	)
 	(segment
-		(start 69.78 62.02)
+		(start 66.5 61.5)
 		(end 67.88 60.12)
 		(width 0.2)
@@
 	)
 	(segment
-		(start 79 64)
-		(end 76.22 61.22)
-		(width 0.2)
-		(layer "F.Cu")
-		(net 28)
-	)
-	(segment
-		(start 71.52 61.22)
+		(start 70.42 62.42)
 		(end 70.42 60.12)
 		(width 0.2)
@@
 	)
 	(segment
-		(start 76.22 61.22)
-		(end 71.52 61.22)
+		(start 71.5 63.5)
+		(end 70.42 62.42)
 		(width 0.2)
 		(layer "F.Cu")
