File: Fiddling with Project 2/05833-Project2.kicad_pcb (KiCad board)
At the start: 2 copper layers, 64.8 x 33.7 mm, 13 parts, among them J1 BB Power, J2 FTDI, J4 GPIO, U1 LM7805, U2 ATmega328-P, Y1 16MHz Resonator

Commit message: solder jumper
Parts:
- added safety pad: SolderJumper_2_Open, Jumper:SolderJumper-2_P1.3mm_Open_RoundedPad1.0x1.5mm, F.Cu at (41.3, 72.4)
Routing:
- net Net-(JP1-A): track 6.37 -> 10.8 mm
- net /DTR: track 81.2 -> 84.8 mm
- added copper zone on B.Cu, net GND
- added copper zone on F.Cu, net GND
Other:
- board size 64.8 x 33.7 mm -> 67.3 x 36.2 mm
- board text added: "Rebekah Julicher"

Commit message: Final touches
Routing:
- net /D6: track 23.1 -> 22.5 mm
Other:
- board text added: "{dblquote}Any sufficiently advanced technology is indistinguishable from magic.{dblquote} -Arthur C. Clarke"
- board text added: "{dblquote}If this doesn't work, I will cry.{dblquote} -Rebekah Julicher"
Changed lines of the file:
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@@
 		(layer "Edge.Cuts")
 	)
-	(gr_text "Rebekah\nJulicher"
-		(at 103.505 81.915 90)
+	(gr_text "{dblquote}If this doesn't work, I will cry.{dblquote}\n-Rebekah Julicher"
+		(at 50.8 72.39 0)
 		(layer "F.SilkS")
 		(effects
@@
 		)
 	)
+	(gr_text "{dblquote}Any sufficiently advanced technology is indistinguishable from magic.{dblquote}\n-Arthur C. Clarke"
+		(at 42.545 52.07 0)
+		(layer "F.SilkS")
+		(effects
+			(font
+				(size 1 1)
+				(thickness 0.15)
+			)
+			(justify left bottom)
+		)
+	)
+	(gr_text "Rebekah\nJulicher"
+		(at 103.505 81.915 90)
+		(layer "F.SilkS")
+		(effects
+			(font
+				(size 0.762 0.762)
+				(thickness 0.15)
+			)
+			(justify left bottom)
+		)
+	)
 	(segment
 		(start 88.265 53.975)
@@
 	)
 	(segment
-		(start 78.105 53.975)
-		(end 77.005 55.075)
-		(width 0.2)
-		(layer "F.Cu")
-		(net 3)
-	)
-	(segment
 		(start 95.25 68.58)
 		(end 99.695 68.58)
@@
 	)
 	(segment
+		(start 62.23 55.245)
+		(end 60.96 53.975)
+		(width 0.2)
+		(layer "F.Cu")
+		(net 3)
+	)
+	(segment
+		(start 78.105 53.975)
+		(end 74.76 53.975)
+		(width 0.2)
+		(layer "F.Cu")
+		(net 3)
+	)
+	(segment
 		(start 96.52 80.01)
 		(end 97.155 79.375)
@@
 	)
 	(segment
-		(start 62.06 55.075)
-		(end 60.96 53.975)
-		(width 0.2)
-		(layer "F.Cu")
-		(net 3)
-	)
-	(segment
 		(start 48.25 64.77)
 		(end 55.91 64.77)
@@
 	)
 	(segment
-		(start 77.005 55.075)
-		(end 62.06 55.075)
-		(width 0.2)
-		(layer "F.Cu")
-		(net 3)
-	)
-	(segment
 		(start 97.155 79.375)
 		(end 97.155 71.12)
@@
 	)
 	(segment
+		(start 74.76 53.975)
+		(end 74.76 54.430635)
+		(width 0.2)
+		(layer "F.Cu")
+		(net 3)
+	)
+	(segment
 		(start 97.155 71.12)
 		(end 99.695 68.58)
@@
 	)
 	(segment
+		(start 74.76 54.430635)
+		(end 73.945635 55.245)
+		(width 0.2)
+		(layer "F.Cu")
+		(net 3)
+	)
+	(segment
 		(start 83.185 53.975)
 		(end 78.105 53.975)
@@
 	)
 	(segment
+		(start 73.945635 55.245)
+		(end 62.23 55.245)
+		(width 0.2)
+		(layer "F.Cu")
+		(net 3)
+	)
+	(segment
 		(start 55.91 61.625)
 		(end 55.88 61.595)
@@
 	)
 	(segment
+		(start 70.52 64.383529)
+		(end 70.52 62.9)
+		(width 0.2)
+		(layer "F.Cu")
+		(net 19)
+	)
+	(segment
 		(start 73.66 64.77)
-		(end 69.215 64.77)
+		(end 70.906471 64.77)
 		(width 0.2)
 		(layer "F.Cu")
@@
 	)
 	(segment
-		(start 68.58 64.135)
+		(start 69.215 61.595)
 		(end 68.58 61.595)
 		(width 0.2)
@@
 	)
 	(segment
-		(start 69.215 64.77)
-		(end 68.58 64.135)
+		(start 70.906471 64.77)
+		(end 70.52 64.383529)
+		(width 0.2)
+		(layer "F.Cu")
+		(net 19)
+	)
+	(segment
+		(start 70.52 62.9)
+		(end 69.215 61.595)
 		(width 0.2)
 		(layer "F.Cu")
@@
 	)
 	(segment
-		(start 66.04 62.865)
-		(end 68.58 65.405)
+		(start 70.12 64.549215)
+		(end 70.975785 65.405)
 		(width 0.2)
 		(layer "F.Cu")
@@
 	)
 	(segment
+		(start 69.85 62.865)
+		(end 70.12 63.135)
+		(width 0.2)
+		(layer "F.Cu")
+		(net 21)
+	)
+	(segment
+		(start 70.975785 65.405)
+		(end 76.2 65.405)
+		(width 0.2)
+		(layer "F.Cu")
+		(net 21)
+	)
+	(segment
+		(start 70.12 63.135)
+		(end 70.12 64.549215)
+		(width 0.2)
+		(layer "F.Cu")
+		(net 21)
+	)
+	(segment
+		(start 66.675 61.595)
+		(end 67.945 62.865)
+		(width 0.2)
+		(layer "F.Cu")
+		(net 21)
+	)
+	(segment
+		(start 67.945 62.865)
+		(end 69.85 62.865)
+		(width 0.2)
+		(layer "F.Cu")
+		(net 21)
+	)
+	(segment
 		(start 66.04 61.595)
-		(end 66.04 62.865)
-		(width 0.2)
-		(layer "F.Cu")
-		(net 21)
-	)
-	(segment
-		(start 68.58 65.405)
-		(end 76.2 65.405)
-		(width 0.2)
-		(layer "F.Cu")
+		(end 66.675 61.595)
+		(width 0.2)
+		(layer "F.Cu")

Commit message: Finished
Parts:
- added D1: LED, LED_THT:LED_D3.0mm, F.Cu at (94.0, 73.7)
- added J3: ISP, 05833:PinHeader_2x03_P2.54mm_Vertical, F.Cu at (78.1, 67.9)
- added R2: R, Resistor_THT:R_Axial_DIN0207_L6.3mm_D2.5mm_P7.62mm_Horizontal, F.Cu at (94.0, 59.1)
- JP1: renamed from safety pad
- moved Y1 1.42 mm to (66.7, 66.0)
- renumbered AREF to AREF1
Connections:
- net Net-(JP1-A) renamed /RESET
Routing:
- net /RESET: track 10.8 -> 45.0 mm
- net +5V: track 89.9 -> 110.0 mm
- net GND: track 89.6 -> 108.1 mm, vias 0 -> 1
- net /D13: track 29.2 -> 46.5 mm, vias 0 -> 1
- net /D12: track 29.2 -> 44.3 mm, vias 0 -> 1
- net /D11: track 29.2 -> 41.3 mm, vias 0 -> 2
- net Net-(D1-A): track 0.00 -> 4.45 mm
- net Net-(U2-XTAL1/PB6): track 3.21 -> 4.74 mm
- net Net-(U2-XTAL2/PB7): track 4.23 -> 5.76 mm
- net /DTR: track 84.8 -> 83.4 mm, vias 2 -> 3
- net /D10: track 29.2 -> 30.1 mm
- net /D6: track 22.5 -> 23.4 mm
- net /D5: track 27.2 -> 28.1 mm
- net /D7: track 21.1 -> 21.9 mm
- net /D9: track 29.2 -> 29.8 mm
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Other:
- board text added: "1"

Commit message: Complete and ordered
Other:
- board text added: "+"
- board text added: "-"
Changed lines of the file:
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@@
+		)
+	)
+	(gr_text "+"
+		(at 95.885 78.105 0)
+		(layer "F.SilkS")
+		(effects
+			(font
+				(size 1 1)
+				(thickness 0.15)
+			)
+			(justify left bottom)
 		)
 	)
@@
 			(font
 				(size 0.635 0.635)
+				(thickness 0.15)
+			)
+			(justify left bottom)
+		)
+	)
+	(gr_text "+"
+		(at 93.345 69.85 0)
+		(layer "F.SilkS")
+		(effects
+			(font
+				(size 1 1)
 				(thickness 0.15)
 			)
@@
 				(thickness 0.15)
 			)
+			(justify left bottom)
+		)
+	)
+	(gr_text "-"
+		(at 93.345 76.2 0)
+		(layer "F.SilkS")
+		(effects
+			(font
+				(size 1 1)
+				(thickness 0.15)
+			)
+			(justify left bottom)
+		)
+	)
+	(gr_text "-"
+		(at 98.425 78.105 0)
+		(layer "F.SilkS")
+		(effects
+			(font
+				(size 1 1)
+				(thickness 0.15)
+			)
