File: Fiddling with Project 2/05833-Project2.kicad_sch (KiCad schematic)
At the start: 13 parts, among them J1 BB Power, J2 FTDI, J3 AREF, J4 GPIO, U1 LM7805, U2 ATmega328-P, Y1 16MHz Resonator

Commit message: Revamped
Parts:
- U1: footprint 05833:TO-220-3_Vertical -> Package_TO_SOT_THT:TO-220-3_Horizontal_TabDown
- renumbered J3 to AREF1
Changed lines of the file:
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@@
 			)
 		)
-		(property "Footprint" "05833:TO-220-3_Vertical"
+		(property "Footprint" "Package_TO_SOT_THT:TO-220-3_Horizontal_TabDown"
 			(at 60.96 20.955 0)
 			(effects
@@
 		(dnp no)
 		(fields_autoplaced yes)
-		(property "Reference" "J3"
+		(property "Reference" "AREF1"
 			(at 88.265 45.72 0)
 			(effects
@@
 			(project "05833-Project2"
 				(path "/e30c0031-f481-430a-8ab4-08825872f914"
-					(reference "J3")
-					(unit 1)
-				)
+					(reference "AREF1")
+					(unit 1)
+				)

Commit message: solder jumper
Parts:
- added JP1: SolderJumper_2_Open, Jumper:SolderJumper-2_P1.3mm_Open_RoundedPad1.0x1.5mm, symbol Jumper:SolderJumper_2_Open
Connections:
- net DTR: now also JP1.2 (B)
- net at C3.1, R1.2, U2.1 (~{RESET}/PC6): now also JP1.1 (A)
Changed lines of the file:
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@@
+	)
+	(junction
+		(at 134.62 99.06)
+		(diameter 0)
+		(color 0 0 0 0)
 	)
 	(junction
@@
 	(wire
 		(pts
+			(xy 147.32 88.9) (xy 147.32 91.44)
+		)
+		(stroke
+			(width 0)
+			(type default)
+		)
+	)
+	(wire
+		(pts
 			(xy 189.23 69.85) (xy 187.96 69.85)
 		)
@@
 	(wire
 		(pts
+			(xy 134.62 99.06) (xy 147.32 99.06)
+		)
+		(stroke
+			(width 0)
+			(type default)
+		)
+	)
+	(wire
+		(pts
 			(xy 125.73 50.8) (xy 127 50.8)
 		)
@@
 		(pts
 			(xy 189.23 90.17) (xy 187.96 90.17)
+		)
+		(stroke
+			(width 0)
+			(type default)
+		)
+	)
+	(wire
+		(pts
+			(xy 147.32 88.9) (xy 134.62 88.9)
 		)
 		(stroke
@@
 					(unit 1)
 				)
+			)
+		)
+	)
+	(symbol
+		(lib_id "Jumper:SolderJumper_2_Open")
+		(at 147.32 95.25 270)
+		(unit 1)
+		(exclude_from_sim no)
+		(in_bom yes)
+		(on_board yes)
+		(dnp no)
+		(fields_autoplaced yes)
+		(property "Reference" "JP1"
+			(at 149.86 93.9799 90)
+			(effects
+				(font
+					(size 1.27 1.27)
+				)
+				(justify left)
+			)
+		)
+		(property "Value" "SolderJumper_2_Open"
+			(at 149.86 96.5199 90)
+			(effects
+				(font
+					(size 1.27 1.27)
+				)
+				(justify left)
+			)
+		)
+		(property "Footprint" "Jumper:SolderJumper-2_P1.3mm_Open_RoundedPad1.0x1.5mm"
+			(at 147.32 95.25 0)
+			(effects
+				(font
+					(size 1.27 1.27)
+				)
+				(hide yes)
+			)
+		)
+		(property "Datasheet" "~"
+			(at 147.32 95.25 0)
+			(effects
+				(font
+					(size 1.27 1.27)
+				)
+				(hide yes)
+			)
+		)
+		(property "Description" "Solder Jumper, 2-pole, open"
+			(at 147.32 95.25 0)
+			(effects
+				(font
+					(size 1.27 1.27)
+				)
+				(hide yes)
+			)
+		)
+		(pin "2"
+		)
+		(pin "1"
+		)
+		(instances
+			(project "05833-Project2"
+				(path "/e30c0031-f481-430a-8ab4-08825872f914"
+					(reference "JP1")
+					(unit 1)
+				)

Commit message: Complete and ordered
Parts:
- added D1: LED, LED_THT:LED_D3.0mm, symbol Device:LED
- added J3: ISP, 05833:PinHeader_2x03_P2.54mm_Vertical, symbol 05833:Conn_02x03_Odd_Even
- added R2: R, Resistor_THT:R_Axial_DIN0207_L6.3mm_D2.5mm_P7.62mm_Horizontal, symbol 05833:R
Connections:
- net +5V: now also J3.2 (Pin_2), R2.1
- net D11: now also J3.4 (Pin_4)
- net D12: now also J3.1 (Pin_1)
- net D13: now also J3.3 (Pin_3)
- net GND: now also D1.1 (K), J3.6 (Pin_6)
- net RESET: now reaches C3.1, JP1.1 (A), R1.2, U2.1 (~{RESET}/PC6)
- net RESET: now also J3.5 (Pin_5)
- new net: D1.2 (A), R2.2
